File: keyboard/kicad/revisions/dormin-rev_1.0/dormin_.kicad_pcb (KiCad board)
At the start: 2 copper layers, 289.7 x 102.8 mm, 202 parts, among them Q1 AO3400A, Q2 AO3407A, Q3_R1 AO3407A, Q4_R1 AO3400A, SW1 SW_Push, SW10 SW_Push, SW11 SW_Push, SW12 SW_Push, SW13 SW_Push, SW14 SW_Push, SW15 SW_Push, SW16 SW_Push, SW17 SW_Push, SW18 SW_Push, SW19 SW_Push, SW2 SW_Push, SW20 SW_Push, SW21 SW_Push, SW22 SW_Push, SW23 SW_Push, SW24 SW_Push, SW25 SW_Push, SW26 SW_Push, SW27 SW_Push, SW28 SW_Push, SW29 SW_Push, SW3 SW_Push, SW30 SW_Push, SW31 SW_Push, SW32 SW_Push, SW33 SW_Push, SW34 SW_Push, SW35 SW_Push, SW36 SW_Push, SW37 SW_Push, SW38 SW_Push, SW39 SW_Push, SW4 SW_Push, SW40 SW_Push, SW5 SW_Push, SW6 SW_Push, SW7 SW_Push, SW8 SW_Push, SW9 SW_Push, U1 XIAO-nRF52840-SMD, U3 XIAO-nRF52840-SMD

Commit message: chore: added temporary routing
Parts:
- added J2: Conn_01x04, Connector_PinSocket_2.54mm:PinSocket_1x04_P2.54mm_Vertical, F.Cu at (77.3, 158.2)
- added J6_R1: Conn_01x04, Connector_PinSocket_2.54mm:PinSocket_1x04_P2.54mm_Vertical, B.Cu at (345.8, 158.2)
- added TP1: VBAT, TestPoint:TestPoint_Pad_D1.0mm, F.Cu at (201.5, 120.5)
- added TP1: VBAT, TestPoint:TestPoint_Pad_D1.0mm, F.Cu at (203.6, 120.4)
- added TP4_R1: VBAT_R, TestPoint:TestPoint_Pad_D1.0mm, B.Cu at (321.2, 144.5)
- added TP6_R1: STS_LED_EN_R, TestPoint:TestPoint_Pad_D1.0mm, B.Cu at (319.4, 159.4)
- moved C7_R1 10.4 mm to (242.9, 120.6), turned to 180 degrees
- moved R715_R1 9.53 mm to (242.9, 122.2)
- moved C8_R1 8.85 mm to (242.9, 118.9), turned to 180 degrees
- moved TP3 1.98 mm to (107.6, 159.4)
Routing:
- net LED_PWM_R: track 206.6 -> 0.00 mm, vias 6 -> 0
- net 3V3_R: track 205.0 -> 2.35 mm, vias 7 -> 0
- net ROW2_R: track 191.5 -> 0.00 mm, vias 12 -> 0
- net ROW1_R: track 169.5 -> 0.00 mm, vias 14 -> 0
- net ROW3_R: track 141.4 -> 0.64 mm, vias 8 -> 0
- net ROW0_R: track 133.6 -> 0.00 mm, vias 7 -> 0
- net RESET_R: track 112.5 -> 6.20 mm, vias 2 -> 0
- net VBAT_R: track 490.4 -> 530.7 mm, vias 6 -> 2
- net SWD: track 0.55 -> 32.5 mm, vias 0 -> 1
- net GND_R: track 18.7 -> 46.2 mm, vias 17 -> 14
- net COL4_R: track 147.2 -> 172.3 mm, vias 4 -> 5
- net Net-(D47_R1-VDD): track 76.1 -> 100.1 mm
- net SWC: track 0.00 -> 23.7 mm, vias 0 -> 2
- net COL2_R: track 185.0 -> 195.6 mm, vias 2 -> 5
- net Net-(D89_R1-A): track 0.00 -> 9.47 mm
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