File: keyboard/kicad/revisions/dormin-rev_1.0/dormin.kicad_pcb (KiCad board)
At the start: 2 copper layers, 289.7 x 102.8 mm, 202 parts, among them Q1 AO3400A, Q2 AO3407A, Q3_R1 AO3407A, Q4_R1 AO3400A, SW1 SW_Push, SW10 SW_Push, SW11 SW_Push, SW12 SW_Push, SW13 SW_Push, SW14 SW_Push, SW15 SW_Push, SW16 SW_Push, SW17 SW_Push, SW18 SW_Push, SW19 SW_Push, SW2 SW_Push, SW20 SW_Push, SW21 SW_Push, SW22 SW_Push, SW23 SW_Push, SW24 SW_Push, SW25 SW_Push, SW26 SW_Push, SW27 SW_Push, SW28 SW_Push, SW29 SW_Push, SW3 SW_Push, SW30 SW_Push, SW31 SW_Push, SW32 SW_Push, SW33 SW_Push, SW34 SW_Push, SW35 SW_Push, SW36 SW_Push, SW37 SW_Push, SW38 SW_Push, SW39 SW_Push, SW4 SW_Push, SW40 SW_Push, SW5 SW_Push, SW6 SW_Push, SW7 SW_Push, SW8 SW_Push, SW9 SW_Push, U1 XIAO-nRF52840-SMD, U3 XIAO-nRF52840-SMD

Commit message: chore: finish main routing
Parts:
- added TP4_R1: VBAT_R, TestPoint:TestPoint_Pad_D1.0mm, B.Cu at (334.2, 139.5)
- added TP6_R1: STS_LED_EN_R, TestPoint:TestPoint_Pad_D1.0mm, B.Cu at (347.1, 156.7)
- moved C1 9.55 mm to (190.1, 110.9), turned to -90 degrees
- moved R712 8.77 mm to (189.2, 113.4)
- moved C2 7.52 mm to (188.3, 110.9), turned to -90 degrees
- turned C4 to 0 degrees
- turned D1 to 180 degrees
Routing:
- net Net-(D21-DIN): track 0.00 -> 133.7 mm, vias 0 -> 2
- net ROW2: track 227.3 -> 193.4 mm, vias 11 -> 13
- net BL_DRAIN: track 429.8 -> 463.2 mm, vias 27 -> 34
- net GND: track 39.3 -> 18.1 mm, vias 12 -> 15
- net VBAT: track 539.8 -> 519.7 mm, vias 4 -> 0
- net COL2: track 154.9 -> 173.4 mm, vias 8 -> 4
- net COL3: track 153.7 -> 171.8 mm, vias 8 -> 7
- net ROW0: track 147.3 -> 133.4 mm, vias 11 -> 14
- net LED_PWM: track 202.4 -> 190.1 mm
- net COL1: track 181.3 -> 193.0 mm
- net ROW3: track 147.8 -> 140.0 mm, vias 13 -> 7
- net VBAT_RAW: track 103.0 -> 96.3 mm, vias 0 -> 2
- net COL4: track 129.6 -> 122.9 mm, vias 10 -> 8
- net COL0: track 194.1 -> 199.2 mm
- net STS_LED_EN: track 150.3 -> 146.4 mm
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- added copper zone on B.Cu, net GND
- added copper zone on F.Cu, net GND
- added copper zone on B.Cu, net GND_R
- added copper zone on F.Cu, net GND_R

Commit message: chore: fix DRC errors
Routing:
- net Net-(D89_R1-A): track 0.00 -> 10.1 mm, vias 0 -> 2
- net Net-(D88_R1-A): track 0.00 -> 9.34 mm
- net ROW1_R: track 169.5 -> 166.1 mm, vias 14 -> 13
- net Net-(D77_R1-K): track 0.00 -> 2.07 mm
- net LED_PWM: track 190.1 -> 189.3 mm
