File: keyboard/kicad/revisions/wolf_keyboard/wlfkbd.kicad_pcb (KiCad board)
At the start: 2 copper layers, 289.7 x 102.8 mm, 204 parts, among them Q1 AO3400A, Q2 AO3407A, Q3_R1 AO3407A, Q4_R1 AO3400A, SW1 SW_Push, SW10 SW_Push, SW11 SW_Push, SW12 SW_Push, SW13 SW_Push, SW14 SW_Push, SW15 SW_Push, SW16 SW_Push, SW17 SW_Push, SW18 SW_Push, SW19 SW_Push, SW2 SW_Push, SW20 SW_Push, SW21 SW_Push, SW22 SW_Push, SW23 SW_Push, SW24 SW_Push, SW25 SW_Push, SW26 SW_Push, SW27 SW_Push, SW28 SW_Push, SW29 SW_Push, SW3 SW_Push, SW30 SW_Push, SW31 SW_Push, SW32 SW_Push, SW33 SW_Push, SW34 SW_Push, SW35 SW_Push, SW36 SW_Push, SW37 SW_Push, SW38 SW_Push, SW39 SW_Push, SW4 SW_Push, SW40 SW_Push, SW5 SW_Push, SW6 SW_Push, SW7 SW_Push, SW8 SW_Push, SW9 SW_Push, U1 XIAO-nRF52840-SMD, U3 XIAO-nRF52840-SMD

Commit message: feat: minor improvements to the routing
Parts:
- moved C5_R1 11.6 mm to (352.8, 102.3)
- moved C6_R1 11.6 mm to (356.1, 102.3)
Routing:
- net GND: track 18.1 -> 20.9 mm, vias 15 -> 16
- net Net-(D47_R1-VDD): track 77.1 -> 79.4 mm
- net Net-(D21-VDD): track 92.3 -> 91.1 mm
- net STS_LED_EN_R: track 172.6 -> 171.9 mm
- net COL1: track 193.0 -> 192.3 mm
- net GND_R: track 18.7 -> 19.2 mm

Commit message: feat: fix schematics after renaming files
Parts:
- BT2_R1: moved to B.Cu
- moved TP1 0.60 mm to (109.4, 147.7)
- moved TP4_R1 0.06 mm to (334.2, 139.4)
Routing:
- net VBAT: track 519.7 -> 523.3 mm
- net Net-(D21-DIN): track 133.4 -> 134.8 mm
- net ROW1: track 155.6 -> 154.7 mm, vias 10 -> 8
- net ROW2: track 193.1 -> 193.2 mm, vias 13 -> 12

Commit message: feat: added test points
Parts:
- added TP2: STS_LED_DATA, TestPoint:TestPoint_Pad_D1.0mm, B.Cu at (189.4, 116.3)
- added TP4: STS_LED_DATA_R, TestPoint:TestPoint_Pad_D1.0mm, B.Cu at (242.9, 115.2)
- added TP5: 3V3_R, TestPoint:TestPoint_Pad_D1.0mm, B.Cu at (346.3, 160.1)
- added TP6: 3V3, TestPoint:TestPoint_Pad_D1.0mm, B.Cu at (82.3, 159.4)
- moved TP6_R1 24.8 mm to (322.4, 158.5)
- moved TP4_R1 23.6 mm to (320.3, 158.5)
- moved TP1 11.9 mm to (111.6, 159.4), turned to 180 degrees
Routing:
- net VBAT_R: track 490.2 -> 528.4 mm, vias 6 -> 8
- net VBAT: track 523.3 -> 537.2 mm
- net 3V3: track 210.7 -> 214.5 mm
- net STS_LED_DATA: track 14.3 -> 17.9 mm
- net STS_LED_EN_R: track 171.9 -> 173.6 mm, vias 4 -> 5
- net STS_LED_DATA_R: track 27.0 -> 28.1 mm
- net 3V3_R: vias 7 -> 8

Commit message: docs: improve README grammar, fixes, and add keyboard repo links
Parts:
- added LOGO1: ~, wlf:Wolf Logo, F.Cu at (307.8, 151.9)
- added LOGO_R1: ~, wlf:Wolf Logo, F.Cu at (122.0, 153.6)
- moved TP2 0.55 mm to (190.0, 116.3)
Routing:
- net STS_LED_DATA: track 17.9 -> 17.4 mm
Other:
- board text added: "Rev 1.0"

Commit message: chore: fix GND plane vias
Parts:
- moved PSW1 0.09 mm to (187.0, 102.8)
- moved PSW2_R1 0.09 mm to (243.0, 102.8)
Routing:
- net GND_R: track 19.2 -> 44.6 mm
- net COL4_R: track 147.2 -> 162.3 mm, vias 4 -> 6
- net VBAT_R: track 528.4 -> 543.1 mm, vias 8 -> 10
- net BL_DRAIN_R: track 435.4 -> 448.4 mm, vias 35 -> 36
- net Net-(D47_R1-DIN): track 127.3 -> 138.9 mm, vias 2 -> 5
- net GND: track 20.9 -> 31.2 mm, vias 16 -> 15
- net Net-(D22-DOUT): track 16.6 -> 21.8 mm, vias 2 -> 3
- net Net-(D23-DOUT): track 16.3 -> 19.3 mm, vias 0 -> 2
- net LED_PWM: track 189.4 -> 186.7 mm
- net COL5_R: track 156.1 -> 153.6 mm, vias 6 -> 8
- net STS_LED_DATA_R: track 28.1 -> 30.5 mm
- net Net-(D47_R1-VDD): track 79.4 -> 81.8 mm, vias 0 -> 4
- net LED_PWM_R: track 206.6 -> 204.6 mm
- net ROW2_R: track 191.5 -> 189.7 mm
- net ROW0_R: track 133.2 -> 131.4 mm
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