File: keyboard/kicad/revisions/wolf_keyboard/wlfkbd.kicad_pcb (KiCad board)
At the start: 2 copper layers, 289.7 x 102.8 mm, 210 parts, among them Q1 AO3400A, Q2 AO3407A, Q3_R1 AO3407A, Q4_R1 AO3400A, SW1 SW_Push, SW10 SW_Push, SW11 SW_Push, SW12 SW_Push, SW13 SW_Push, SW14 SW_Push, SW15 SW_Push, SW16 SW_Push, SW17 SW_Push, SW18 SW_Push, SW19 SW_Push, SW2 SW_Push, SW20 SW_Push, SW21 SW_Push, SW22 SW_Push, SW23 SW_Push, SW24 SW_Push, SW25 SW_Push, SW26 SW_Push, SW27 SW_Push, SW28 SW_Push, SW29 SW_Push, SW3 SW_Push, SW30 SW_Push, SW31 SW_Push, SW32 SW_Push, SW33 SW_Push, SW34 SW_Push, SW35 SW_Push, SW36 SW_Push, SW37 SW_Push, SW38 SW_Push, SW39 SW_Push, SW4 SW_Push, SW40 SW_Push, SW5 SW_Push, SW6 SW_Push, SW7 SW_Push, SW8 SW_Push, SW9 SW_Push, U1 XIAO-nRF52840-SMD, U3 XIAO-nRF52840-SMD

Commit message: chore: fix traces and orgaize schematics
Parts:
- moved TP5 1.60 mm to (346.3, 158.5)
Routing:
- net 3V3_R: track 204.8 -> 207.0 mm
- net VBAT: track 538.0 -> 536.7 mm
- net Net-(D21-VDD): track 92.6 -> 91.4 mm

Commit message: chore: update schematics
Connections:
- U1 pad 15: SWD_R -> unconnected-(U1-SWDIO-Pad15)
- U1 pad 16: SWC_R -> unconnected-(U1-SWCLK-Pad16)
- U3 pad 15: SWD -> unconnected-(U3-SWDIO-Pad15)
- U3 pad 16: SWC -> unconnected-(U3-SWCLK-Pad16)
Changed lines of the file:
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@@
 		(capping no)
 		(filling no)
+		(zone_defaults)
 		(grid_origin 242.78 102.5025)
 		(pcbplotparams
@@
 			(size 1.7 1.7)
 			(layers "B.Cu" "B.Mask" "B.Paste")
-			(net "SWD_R")
+			(net "unconnected-(U1-SWDIO-Pad15)")
 			(pinfunction "SWDIO_15")
-			(pintype "passive")
+			(pintype "passive+no_connect")
 		)
 		(pad "16" smd circle
@@
 			(size 1.7 1.7)
 			(layers "B.Cu" "B.Mask" "B.Paste")
-			(net "SWC_R")
+			(net "unconnected-(U1-SWCLK-Pad16)")
 			(pinfunction "SWCLK_16")
-			(pintype "passive")
+			(pintype "passive+no_connect")
 		)
 		(pad "17" smd circle
@@
 			(size 1.7 1.7)
 			(layers "B.Cu" "B.Mask" "B.Paste")
-			(net "SWD")
+			(net "unconnected-(U3-SWDIO-Pad15)")
 			(pinfunction "SWDIO_15")
-			(pintype "passive")
+			(pintype "passive+no_connect")
 		)
 		(pad "16" smd circle
@@
 			(size 1.7 1.7)
 			(layers "B.Cu" "B.Mask" "B.Paste")
-			(net "SWC")
+			(net "unconnected-(U3-SWCLK-Pad16)")
 			(pinfunction "SWCLK_16")
-			(pintype "passive")
+			(pintype "passive+no_connect")
 		)
 		(pad "17" smd circle

Commit message: feat: added mousebites
Parts:
- added REF**: BreakLine_5h_D0.5mm_P0.85mm, Panelization:BreakLine_5h_D0.5mm_P0.85mm, F.Cu at (272.2, 96.3)
- added REF**: BreakLine_5h_D0.5mm_P0.85mm, Panelization:BreakLine_5h_D0.5mm_P0.85mm, F.Cu at (118.4, 96.3)
- added REF**: BreakLine_5h_D0.5mm_P0.85mm, Panelization:BreakLine_5h_D0.5mm_P0.85mm, F.Cu at (157.9, 96.3)
- added REF**: BreakLine_5h_D0.5mm_P0.85mm, Panelization:BreakLine_5h_D0.5mm_P0.85mm, F.Cu at (311.7, 96.3)
Routing:
- net VBAT: track 536.7 -> 536.2 mm
- net ROW0: track 133.1 -> 133.6 mm
- net LED_PWM: track 186.7 -> 186.2 mm
Other:
- board size 289.7 x 102.8 mm -> 289.7 x 109.2 mm

Commit message: feat: added production files
Parts:
- SW1, SW10, SW11, SW12, SW13, SW14, SW15, SW16, SW17, SW18, SW19, SW2, SW20, SW21, SW22, SW23, SW24, SW25, SW26, SW27, SW28, SW29, SW3, SW30, SW31, SW32, SW33, SW34, SW35, SW36, SW37, SW38, SW39, SW4, SW40, SW5, SW6, SW7, SW8, SW9: footprint willkeebs_keyboard:NF_LED_1206_SW_KS33_3_0_HS_1U -> willkeebs_keyboard:KS-33B Hotswap 1u; moved to B.Cu
