File: keyboard/kicad/revisions/wolf_keyboard/wlfkbd_left.kicad_sch (KiCad schematic)
At the start: 102 parts, among them Q1 AO3400A, Q2 AO3407A, SW1 SW_Push, SW10 SW_Push, SW11 SW_Push, SW12 SW_Push, SW13 SW_Push, SW14 SW_Push, SW15 SW_Push, SW16 SW_Push, SW17 SW_Push, SW18 SW_Push, SW19 SW_Push, SW2 SW_Push, SW20 SW_Push, SW3 SW_Push, SW4 SW_Push, SW5 SW_Push, SW6 SW_Push, SW7 SW_Push, SW8 SW_Push, SW9 SW_Push, U3 XIAO-nRF52840-SMD

Commit message: feat: added test points
Parts:
- added TP2: STS_LED_DATA, TestPoint:TestPoint_Pad_D1.0mm, symbol Connector:TestPoint
- added TP6: 3V3, TestPoint:TestPoint_Pad_D1.0mm, symbol Connector:TestPoint
Connections:
- net 3V3: now also TP6.1
- net STS_LED_DATA: now also TP2.1
Other:
- note added: "W O L F K B D"
- note removed: "D O R M I N"
- moved on the sheet: TP1, TP3, U3

Commit message: docs: improve README grammar, fixes, and add keyboard repo links
Parts:
- added LOGO1: (no value), wlf:Wolf Logo, symbol wlf:wlf_logo
Other:
- note added: "LOGO"
Changed lines of the file:
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@@
 		)
 	)
+	(text "LOGO"
+		(exclude_from_sim no)
+		(at 143.51 185.42 0)
+		(effects
+			(font
+				(size 2 2)
+			)
+			(justify left bottom)
+		)
+	)
 	(text "MCU"
 		(exclude_from_sim no)
@@
 					(unit 1)
 				)
+			)
+		)
+	)
+	(symbol
+		(lib_id "wlf:wlf_logo")
+		(at 147.32 193.04 0)
+		(unit 1)
+		(body_style 1)
+		(exclude_from_sim no)
+		(in_bom yes)
+		(on_board yes)
+		(in_pos_files yes)
+		(dnp no)
+		(property "Reference" "LOGO1"
+			(at 147.32 189.23 0)
+			(hide yes)
+			(show_name no)
+			(do_not_autoplace no)
+			(effects
+				(font
+					(size 1.27 1.27)
+				)
+			)
+		)
+		(property "Value" ""
+			(at 147.32 193.04 0)
+			(show_name no)
+			(do_not_autoplace no)
+			(effects
+				(font
+					(size 1.27 1.27)
+				)
+			)
+		)
+		(property "Footprint" "wlf:Wolf Logo"
+			(at 149.86 195.58 0)
+			(show_name no)
+			(do_not_autoplace no)
+			(effects
+				(font
+					(size 1.27 1.27)
+				)
+			)
+		)
+		(property "Datasheet" ""
+			(at 147.32 193.04 0)
+			(hide yes)
+			(show_name no)
+			(do_not_autoplace no)
+			(effects
+				(font
+					(size 1.27 1.27)
+				)
+			)
+		)
+		(property "Description" ""
+			(at 147.32 193.04 0)
+			(hide yes)
+			(show_name no)
+			(do_not_autoplace no)
+			(effects
+				(font
+					(size 1.27 1.27)
+				)
+			)
+		)
+		(instances
+			(project "wlfkbd"
+				(path "/603afaa0-4142-4673-b835-76ba767ab9eb/61f422a6-c5c1-4994-83bd-f5d919e1e268"
+					(reference "LOGO1")
+					(unit 1)
+				)

Commit message: chore: fix traces and orgaize schematics
Connections:
- net SWC: no longer names the net of U3.16 (SWCLK)
- net SWD: no longer names the net of U3.15 (SWDIO)
- no-connect marks 3 -> 5
Changed lines of the file:
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@@
 	(text "W O L F K B D"
 		(exclude_from_sim no)
-		(at 10.16 234.95 0)
+		(at 11.43 234.95 0)
 		(effects
 			(font
@@
 	(text "MCU"
 		(exclude_from_sim no)
-		(at 63.5 29.21 0)
+		(at 63.5 22.86 0)
 		(effects
 			(font
@@
 	)
 	(no_connect
+		(at 91.44 40.64)
+	)
+	(no_connect
+		(at 87.63 40.64)
+	)
+	(no_connect
 		(at 111.76 48.26)
 	)
@@
 	(polyline
 		(pts
-			(xy 12.7 167.64) (xy 176.53 166.37)
+			(xy 12.7 167.64) (xy 179.07 166.37)
 		)
 		(stroke
@@
 	(polyline
 		(pts
-			(xy 176.53 13.97) (xy 177.8 241.3)
+			(xy 179.07 12.7) (xy 180.34 240.03)
 		)
 		(stroke
@@
 	(polyline
 		(pts
-			(xy 13.97 209.55) (xy 176.53 209.55)
+			(xy 13.97 209.55) (xy 179.07 209.55)
 		)
 		(stroke
@@
 		)
 	)
-	(global_label "SWC"
-		(shape input)
-		(at 91.44 40.64 90)
-		(fields_autoplaced yes)
-		(effects
-			(font
-				(size 1.27 1.27)
-			)
-			(justify left)
-		)
-		(property "Intersheetrefs" "${INTERSHEET_REFS}"
-			(at 91.44 33.7239 90)
-			(hide yes)
-			(show_name no)
-			(do_not_autoplace no)
-			(effects
-				(font
-					(size 1.27 1.27)
-				)
-				(justify left)
-			)
-		)
-	)
 	(global_label "STS_LED_EN"
 		(shape input)
@@
 		)
 	)
-	(global_label "SWD"
-		(shape input)
-		(at 87.63 40.64 90)
-		(fields_autoplaced yes)
-		(effects
-			(font
-				(size 1.27 1.27)
-			)
-			(justify left)
-		)
-		(property "Intersheetrefs" "${INTERSHEET_REFS}"
-			(at 87.63 33.7239 90)
-			(hide yes)
-			(show_name no)
-			(do_not_autoplace no)
-			(effects
-				(font
-					(size 1.27 1.27)
-				)
-				(justify left)
-			)
-		)
-	)
 	(global_label "LED_PWM"
 		(shape input)
@@
 		(in_pos_files yes)
 		(dnp no)
-		(fields_autoplaced yes)
 		(property "Reference" "U3"
-			(at 101.2033 38.1 0)
+			(at 63.5 25.4 0)
 			(show_name no)
 			(do_not_autoplace no)
@@
 		)
 		(property "Value" "XIAO-nRF52840-SMD"
-			(at 101.2033 40.64 0)
+			(at 63.5 27.94 0)
 			(show_name no)
 			(do_not_autoplace no)

Commit message: feat: added production files
Parts:
- SW1, SW10, SW11, SW12, SW13, SW14, SW15, SW16, SW17, SW18, SW19, SW2, SW20, SW3, SW4, SW5, SW6, SW7, SW8, SW9: footprint willkeebs_keyboard:NF_LED_1206_SW_KS33_3_0_HS_1U -> willkeebs_keyboard:KS-33B Hotswap 1u
Changed lines of the file:
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@@
 			)
 		)
-		(property "Footprint" "willkeebs_keyboard:NF_LED_1206_SW_KS33_3_0_HS_1U"
+		(property "Footprint" "willkeebs_keyboard:KS-33B Hotswap 1u"
 			(at 208.28 60.96 0)
 			(hide yes)
@@
 			)
 		)
-		(property "Footprint" "willkeebs_keyboard:NF_LED_1206_SW_KS33_3_0_HS_1U"
+		(property "Footprint" "willkeebs_keyboard:KS-33B Hotswap 1u"
 			(at 266.7 91.44 0)
 			(hide yes)
@@
 			)
 		)
-		(property "Footprint" "willkeebs_keyboard:NF_LED_1206_SW_KS33_3_0_HS_1U"
+		(property "Footprint" "willkeebs_keyboard:KS-33B Hotswap 1u"
 			(at 223.52 76.2 0)
 			(hide yes)
@@
 			)
 		)
-		(property "Footprint" "willkeebs_keyboard:NF_LED_1206_SW_KS33_3_0_HS_1U"
+		(property "Footprint" "willkeebs_keyboard:KS-33B Hotswap 1u"
 			(at 251.46 76.2 0)
 			(hide yes)
@@
 			)
 		)
-		(property "Footprint" "willkeebs_keyboard:NF_LED_1206_SW_KS33_3_0_HS_1U"
+		(property "Footprint" "willkeebs_keyboard:KS-33B Hotswap 1u"
 			(at 223.52 60.96 0)
 			(hide yes)
@@
 			)
 		)
-		(property "Footprint" "willkeebs_keyboard:NF_LED_1206_SW_KS33_3_0_HS_1U"
+		(property "Footprint" "willkeebs_keyboard:KS-33B Hotswap 1u"
 			(at 266.7 60.96 0)
 			(hide yes)
@@
 			)
 		)
-		(property "Footprint" "willkeebs_keyboard:NF_LED_1206_SW_KS33_3_0_HS_1U"
+		(property "Footprint" "willkeebs_keyboard:KS-33B Hotswap 1u"
 			(at 223.52 45.72 0)
 			(hide yes)
@@
 			)
 		)
-		(property "Footprint" "willkeebs_keyboard:NF_LED_1206_SW_KS33_3_0_HS_1U"
+		(property "Footprint" "willkeebs_keyboard:KS-33B Hotswap 1u"
 			(at 237.49 76.2 0)
 			(hide yes)
@@
 			)
 		)
-		(property "Footprint" "willkeebs_keyboard:NF_LED_1206_SW_KS33_3_0_HS_1U"
+		(property "Footprint" "willkeebs_keyboard:KS-33B Hotswap 1u"
 			(at 281.94 76.2 0)
 			(hide yes)
@@
 			)
 		)
-		(property "Footprint" "willkeebs_keyboard:NF_LED_1206_SW_KS33_3_0_HS_1U"
+		(property "Footprint" "willkeebs_keyboard:KS-33B Hotswap 1u"
 			(at 251.46 45.72 0)
 			(hide yes)
@@
 			)
 		)
-		(property "Footprint" "willkeebs_keyboard:NF_LED_1206_SW_KS33_3_0_HS_1U"
+		(property "Footprint" "willkeebs_keyboard:KS-33B Hotswap 1u"
 			(at 251.46 91.44 0)
 			(hide yes)
@@
 			)
 		)
-		(property "Footprint" "willkeebs_keyboard:NF_LED_1206_SW_KS33_3_0_HS_1U"
+		(property "Footprint" "willkeebs_keyboard:KS-33B Hotswap 1u"
 			(at 237.49 45.72 0)
 			(hide yes)
@@
 			)
 		)
-		(property "Footprint" "willkeebs_keyboard:NF_LED_1206_SW_KS33_3_0_HS_1U"
+		(property "Footprint" "willkeebs_keyboard:KS-33B Hotswap 1u"
 			(at 251.46 60.96 0)
 			(hide yes)
@@
 			)
 		)
-		(property "Footprint" "willkeebs_keyboard:NF_LED_1206_SW_KS33_3_0_HS_1U"
+		(property "Footprint" "willkeebs_keyboard:KS-33B Hotswap 1u"
 			(at 281.94 91.44 0)
 			(hide yes)
@@
 			)
 		)
-		(property "Footprint" "willkeebs_keyboard:NF_LED_1206_SW_KS33_3_0_HS_1U"
+		(property "Footprint" "willkeebs_keyboard:KS-33B Hotswap 1u"
 			(at 208.28 76.2 0)
 			(hide yes)
@@
 			)
 		)
-		(property "Footprint" "willkeebs_keyboard:NF_LED_1206_SW_KS33_3_0_HS_1U"
+		(property "Footprint" "willkeebs_keyboard:KS-33B Hotswap 1u"
 			(at 266.7 45.72 0)
 			(hide yes)
@@
 			)
 		)
-		(property "Footprint" "willkeebs_keyboard:NF_LED_1206_SW_KS33_3_0_HS_1U"
+		(property "Footprint" "willkeebs_keyboard:KS-33B Hotswap 1u"
 			(at 237.49 60.96 0)
 			(hide yes)
@@
 			)
 		)
-		(property "Footprint" "willkeebs_keyboard:NF_LED_1206_SW_KS33_3_0_HS_1U"
+		(property "Footprint" "willkeebs_keyboard:KS-33B Hotswap 1u"
 			(at 266.7 76.2 0)
 			(hide yes)
@@
 			)
 		)
-		(property "Footprint" "willkeebs_keyboard:NF_LED_1206_SW_KS33_3_0_HS_1U"
+		(property "Footprint" "willkeebs_keyboard:KS-33B Hotswap 1u"
 			(at 281.94 45.72 0)
 			(hide yes)
@@
 			)
 		)
-		(property "Footprint" "willkeebs_keyboard:NF_LED_1206_SW_KS33_3_0_HS_1U"
+		(property "Footprint" "willkeebs_keyboard:KS-33B Hotswap 1u"
 			(at 281.94 60.96 0)
 			(hide yes)

Commit message: feat: remove unused components from BOM and POS
Parts:
- BT1, TP1, TP2, TP3, TP6: now left out of the parts list
Changed lines of the file:
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@@
 		(body_style 1)
 		(exclude_from_sim no)
-		(in_bom yes)
+		(in_bom no)
 		(on_board yes)
-		(in_pos_files yes)
+		(in_pos_files no)
 		(dnp no)
 		(property "Reference" "TP1"
@@
 		(body_style 1)
 		(exclude_from_sim no)
-		(in_bom yes)
+		(in_bom no)
 		(on_board yes)
-		(in_pos_files yes)
+		(in_pos_files no)
 		(dnp no)
 		(property "Reference" "TP3"
@@
 		(body_style 1)
 		(exclude_from_sim no)
-		(in_bom yes)
+		(in_bom no)
 		(on_board yes)
-		(in_pos_files yes)
+		(in_pos_files no)
 		(dnp no)
 		(property "Reference" "TP2"
@@
 		(body_style 1)
 		(exclude_from_sim no)
-		(in_bom yes)
+		(in_bom no)
 		(on_board yes)
-		(in_pos_files yes)
+		(in_pos_files no)
 		(dnp no)
 		(property "Reference" "BT1"
@@
 		(body_style 1)
 		(exclude_from_sim no)
-		(in_bom yes)
+		(in_bom no)
 		(on_board yes)
-		(in_pos_files yes)
+		(in_pos_files no)
 		(dnp no)
 		(fields_autoplaced yes)

Commit message: feat: remove unused components from BOM and POS
Parts:
- LOGO1: now left out of the parts list
Changed lines of the file:
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@@
 		(body_style 1)
 		(exclude_from_sim no)
-		(in_bom yes)
+		(in_bom no)
 		(on_board yes)
-		(in_pos_files yes)
+		(in_pos_files no)
 		(dnp no)
 		(property "Reference" "LOGO1"
