File: keyboard/kicad/revisions/wolf_keyboard/wlfkbd_right.kicad_sch (KiCad schematic)
At the start: 102 parts, among them Q3_R1 AO3407A, Q4_R1 AO3400A, SW21 SW_Push, SW22 SW_Push, SW23 SW_Push, SW24 SW_Push, SW25 SW_Push, SW26 SW_Push, SW27 SW_Push, SW28 SW_Push, SW29 SW_Push, SW30 SW_Push, SW31 SW_Push, SW32 SW_Push, SW33 SW_Push, SW34 SW_Push, SW35 SW_Push, SW36 SW_Push, SW37 SW_Push, SW38 SW_Push, SW39 SW_Push, SW40 SW_Push, U1 XIAO-nRF52840-SMD

Commit message: feat: added test points
Parts:
- added TP4: STS_LED_DATA_R, TestPoint:TestPoint_Pad_D1.0mm, symbol Connector:TestPoint
- added TP5: 3V3_R, TestPoint:TestPoint_Pad_D1.0mm, symbol Connector:TestPoint
Connections:
- net 3V3_R: now also TP5.1
- net STS_LED_DATA_R: now also TP4.1
Other:
- note added: "W O L F K B D"
- note removed: "D O R M I N"
- moved on the sheet: TP4_R1, TP6_R1, U1

Commit message: docs: improve README grammar, fixes, and add keyboard repo links
Parts:
- added LOGO_R1: (no value), wlf:Wolf Logo, symbol wlf:wlf_logo
Other:
- note added: "LOGO"
Changed lines of the file:
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@@
 		)
 	)
+	(text "LOGO"
+		(exclude_from_sim no)
+		(at 154.94 184.15 0)
+		(effects
+			(font
+				(size 2 2)
+			)
+			(justify left bottom)
+		)
+	)
 	(text "Place Capacitors\nnear the first LED in chain (PCB)"
 		(exclude_from_sim no)
@@
 					(unit 1)
 				)
+			)
+		)
+	)
+	(symbol
+		(lib_id "wlf:wlf_logo")
+		(at 158.75 194.31 0)
+		(unit 1)
+		(body_style 1)
+		(exclude_from_sim no)
+		(in_bom yes)
+		(on_board yes)
+		(in_pos_files yes)
+		(dnp no)
+		(fields_autoplaced yes)
+		(property "Reference" "LOGO_R1"
+			(at 158.75 190.5 0)
+			(hide yes)
+			(show_name no)
+			(do_not_autoplace no)
+			(effects
+				(font
+					(size 1.27 1.27)
+				)
+			)
+		)
+		(property "Value" ""
+			(at 158.75 194.31 0)
+			(show_name no)
+			(do_not_autoplace no)
+			(effects
+				(font
+					(size 1.27 1.27)
+				)
+			)
+		)
+		(property "Footprint" "wlf:Wolf Logo"
+			(at 158.75 194.31 0)
+			(hide yes)
+			(show_name no)
+			(do_not_autoplace no)
+			(effects
+				(font
+					(size 1.27 1.27)
+				)
+			)
+		)
+		(property "Datasheet" ""
+			(at 158.75 194.31 0)
+			(hide yes)
+			(show_name no)
+			(do_not_autoplace no)
+			(effects
+				(font
+					(size 1.27 1.27)
+				)
+			)
+		)
+		(property "Description" ""
+			(at 158.75 194.31 0)
+			(hide yes)
+			(show_name no)
+			(do_not_autoplace no)
+			(effects
+				(font
+					(size 1.27 1.27)
+				)
+			)
+		)
+		(instances
+			(project "wlfkbd"
+				(path "/603afaa0-4142-4673-b835-76ba767ab9eb/c34ad971-40ee-4ba1-b588-4be495453fb3"
+					(reference "LOGO_R1")
+					(unit 1)
+				)

Commit message: chore: fix traces and orgaize schematics
Changed lines of the file:
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@@
 	(text "W O L F K B D"
 		(exclude_from_sim no)
-		(at 10.16 237.49 0)
+		(at 11.43 237.49 0)
 		(effects
 			(font
@@
 	(text "MCU"
 		(exclude_from_sim no)
-		(at 59.69 22.86 0)
+		(at 57.15 19.05 0)
 		(effects
 			(font
@@
 	(polyline
 		(pts
-			(xy 176.53 13.97) (xy 177.8 241.3)
+			(xy 179.07 13.97) (xy 180.34 241.3)
 		)
 		(stroke
@@
 	(polyline
 		(pts
-			(xy 12.7 167.64) (xy 176.53 166.37)
+			(xy 12.7 167.64) (xy 179.07 166.37)
 		)
 		(stroke
@@
 	(polyline
 		(pts
-			(xy 13.97 209.55) (xy 176.53 209.55)
+			(xy 12.7 209.55) (xy 179.07 209.55)
 		)
 		(stroke
@@
 		(in_pos_files yes)
 		(dnp no)
-		(fields_autoplaced yes)
 		(property "Reference" "U1"
-			(at 94.8533 35.56 0)
+			(at 57.15 21.59 0)
 			(show_name no)
 			(do_not_autoplace no)
@@
 		)
 		(property "Value" "XIAO-nRF52840-SMD"
-			(at 94.8533 38.1 0)
+			(at 57.15 24.13 0)
 			(show_name no)
 			(do_not_autoplace no)

Commit message: chore: update schematics
Connections:
- net SWC_R: no longer names the net of U1.16 (SWCLK)
- net SWD_R: no longer names the net of U1.15 (SWDIO)
- no-connect marks 3 -> 5
Changed lines of the file:
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@@
+	)
+	(no_connect
+		(at 85.09 38.1)
 	)
 	(no_connect
@@
 	)
 	(no_connect
+		(at 81.28 38.1)
+	)
+	(no_connect
 		(at 156.21 140.97)
 	)
@@
 		)
 	)
-	(global_label "SWC_R"
-		(shape input)
-		(at 85.09 38.1 90)
+	(global_label "COL2_R"
+		(shape input)
+		(at 67.31 68.58 180)
+		(fields_autoplaced yes)
+		(effects
+			(font
+				(size 1.27 1.27)
+			)
+			(justify right)
+		)
+		(property "Intersheetrefs" "${INTERSHEET_REFS}"
+			(at 57.2491 68.58 0)
+			(hide yes)
+			(show_name no)
+			(do_not_autoplace no)
+			(effects
+				(font
+					(size 1.27 1.27)
+				)
+				(justify right)
+			)
+		)
+	)
+	(global_label "ROW2_R"
+		(shape input)
+		(at 67.31 53.34 180)
+		(fields_autoplaced yes)
+		(effects
+			(font
+				(size 1.27 1.27)
+			)
+			(justify right)
+		)
+		(property "Intersheetrefs" "${INTERSHEET_REFS}"
+			(at 56.8258 53.34 0)
+			(hide yes)
+			(show_name no)
+			(do_not_autoplace no)
+			(effects
+				(font
+					(size 1.27 1.27)
+				)
+				(justify right)
+			)
+		)
+	)
+	(global_label "BL_DRAIN_R"
+		(shape input)
+		(at 287.02 152.4 180)
+		(fields_autoplaced yes)
+		(effects
+			(font
+				(size 1.27 1.27)
+			)
+			(justify right)
+		)
+		(property "Intersheetrefs" "${INTERSHEET_REFS}"
+			(at 275.2052 152.4 0)
+			(hide yes)
+			(show_name no)
+			(do_not_autoplace no)
+			(effects
+				(font
+					(size 1.27 1.27)
+				)
+				(justify right)
+			)
+		)
+	)
+	(global_label "COL0_R"
+		(shape input)
+		(at 67.31 60.96 180)
+		(fields_autoplaced yes)
+		(effects
+			(font
+				(size 1.27 1.27)
+			)
+			(justify right)
+		)
+		(property "Intersheetrefs" "${INTERSHEET_REFS}"
+			(at 59.4867 60.96 0)
+			(hide yes)
+			(show_name no)
+			(do_not_autoplace no)
+			(effects
+				(font
+					(size 1.27 1.27)
+				)
+				(justify right)
+			)
+		)
+	)
+	(global_label "RESET_R"
+		(shape input)
+		(at 88.9 38.1 90)
 		(fields_autoplaced yes)
 		(effects
@@
 		)
 		(property "Intersheetrefs" "${INTERSHEET_REFS}"
-			(at 85.09 31.1839 90)
+			(at 88.9 29.3697 90)
 			(hide yes)
 			(show_name no)
@@
 		)
 	)
-	(global_label "COL2_R"
-		(shape input)
-		(at 67.31 68.58 180)
+	(global_label "STS_LED_DATA_R"
+		(shape input)
+		(at 87.63 151.13 180)
 		(fields_autoplaced yes)
 		(effects
@@
 		)
 		(property "Intersheetrefs" "${INTERSHEET_REFS}"
-			(at 57.2491 68.58 0)
+			(at 71.4611 151.13 0)
 			(hide yes)
 			(show_name no)
@@
 		)
 	)
-	(global_label "ROW2_R"
-		(shape input)
-		(at 67.31 53.34 180)
+	(global_label "COL4_R"
+		(shape input)
+		(at 278.13 36.83 90)
+		(fields_autoplaced yes)
+		(effects
+			(font
+				(size 1.27 1.27)
+			)
+			(justify left)
+		)
+		(property "Intersheetrefs" "${INTERSHEET_REFS}"
+			(at 278.13 29.0067 90)
+			(hide yes)
+			(show_name no)
+			(do_not_autoplace no)
+			(effects
+				(font
+					(size 1.27 1.27)
+				)
+				(justify left)
+			)
+		)
+	)
+	(global_label "VBAT_RAW_R"
+		(shape input)
+		(at 88.9 186.69 270)
 		(fields_autoplaced yes)
 		(effects
@@
 		)
 		(property "Intersheetrefs" "${INTERSHEET_REFS}"
-			(at 56.8258 53.34 0)
+			(at 88.9 198.8676 90)
 			(hide yes)
 			(show_name no)
@@
 		)
 	)
-	(global_label "BL_DRAIN_R"
-		(shape input)
-		(at 287.02 152.4 180)
+	(global_label "ROW0_R"
+		(shape input)
+		(at 67.31 45.72 180)
 		(fields_autoplaced yes)
 		(effects
@@
 		)
 		(property "Intersheetrefs" "${INTERSHEET_REFS}"
-			(at 275.2052 152.4 0)
+			(at 56.8258 45.72 0)
 			(hide yes)
 			(show_name no)
@@
 			)
 		)
-	)
-	(global_label "COL0_R"
-		(shape input)
-		(at 67.31 60.96 180)
-		(fields_autoplaced yes)
-		(effects
-			(font
-				(size 1.27 1.27)
-			)
-			(justify right)
-		)
-		(property "Intersheetrefs" "${INTERSHEET_REFS}"
-			(at 59.4867 60.96 0)
-			(hide yes)
-			(show_name no)
-			(do_not_autoplace no)
-			(effects
-				(font
-					(size 1.27 1.27)
-				)
-				(justify right)
-			)
-		)
-	)
-	(global_label "RESET_R"
-		(shape input)
-		(at 88.9 38.1 90)
-		(fields_autoplaced yes)
-		(effects
-			(font
-				(size 1.27 1.27)
-			)
-			(justify left)
-		)
-		(property "Intersheetrefs" "${INTERSHEET_REFS}"
-			(at 88.9 29.3697 90)
-			(hide yes)
-			(show_name no)
-			(do_not_autoplace no)
-			(effects
-				(font
-					(size 1.27 1.27)
-				)
-				(justify left)
-			)
-		)
-	)
-	(global_label "STS_LED_DATA_R"
-		(shape input)
-		(at 87.63 151.13 180)
-		(fields_autoplaced yes)
-		(effects
-			(font
-				(size 1.27 1.27)
-			)
-			(justify right)
-		)
-		(property "Intersheetrefs" "${INTERSHEET_REFS}"
-			(at 71.4611 151.13 0)
-			(hide yes)
-			(show_name no)
-			(do_not_autoplace no)
-			(effects
-				(font
-					(size 1.27 1.27)
-				)
-				(justify right)
-			)
-		)
-	)
-	(global_label "COL4_R"
-		(shape input)
-		(at 278.13 36.83 90)
-		(fields_autoplaced yes)
-		(effects
-			(font
-				(size 1.27 1.27)
-			)
-			(justify left)
-		)
-		(property "Intersheetrefs" "${INTERSHEET_REFS}"
-			(at 278.13 29.0067 90)
-			(hide yes)
-			(show_name no)
-			(do_not_autoplace no)
-			(effects
-				(font
-					(size 1.27 1.27)
-				)
-				(justify left)
-			)
-		)
-	)
-	(global_label "VBAT_RAW_R"
-		(shape input)
-		(at 88.9 186.69 270)
-		(fields_autoplaced yes)
-		(effects
-			(font
-				(size 1.27 1.27)
-			)
-			(justify right)
-		)
-		(property "Intersheetrefs" "${INTERSHEET_REFS}"
-			(at 88.9 198.8676 90)
-			(hide yes)
-			(show_name no)
-			(do_not_autoplace no)
-			(effects
-				(font
-					(size 1.27 1.27)
-				)
-				(justify right)
-			)
-		)
-	)
-	(global_label "ROW0_R"
-		(shape input)
-		(at 67.31 45.72 180)
-		(fields_autoplaced yes)
-		(effects
-			(font
-				(size 1.27 1.27)
-			)
-			(justify right)
-		)
-		(property "Intersheetrefs" "${INTERSHEET_REFS}"
-			(at 56.8258 45.72 0)
-			(hide yes)
-			(show_name no)
-			(do_not_autoplace no)
-			(effects
-				(font
-					(size 1.27 1.27)
-				)
-				(justify right)
-			)
-		)
-	)
-	(global_label "SWD_R"
-		(shape input)
-		(at 81.28 38.1 90)
-		(fields_autoplaced yes)
-		(effects
-			(font
-				(size 1.27 1.27)
-			)
-			(justify left)
-		)
-		(property "Intersheetrefs" "${INTERSHEET_REFS}"
-			(at 81.28 31.1839 90)
-			(hide yes)
-			(show_name no)
-			(do_not_autoplace no)
-			(effects
-				(font
-					(size 1.27 1.27)
-				)
-				(justify left)
-			)
-		)

Commit message: feat: added production files
Parts:
- SW21, SW22, SW23, SW24, SW25, SW26, SW27, SW28, SW29, SW30, SW31, SW32, SW33, SW34, SW35, SW36, SW37, SW38, SW39, SW40: footprint willkeebs_keyboard:NF_LED_1206_SW_KS33_3_0_HS_1U -> willkeebs_keyboard:KS-33B Hotswap 1u
Changed lines of the file:
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@@
 			)
 		)
-		(property "Footprint" "willkeebs_keyboard:NF_LED_1206_SW_KS33_3_0_HS_1U"
+		(property "Footprint" "willkeebs_keyboard:KS-33B Hotswap 1u"
 			(at 231.14 41.91 0)
 			(hide yes)
@@
 			)
 		)
-		(property "Footprint" "willkeebs_keyboard:NF_LED_1206_SW_KS33_3_0_HS_1U"
+		(property "Footprint" "willkeebs_keyboard:KS-33B Hotswap 1u"
 			(at 259.08 57.15 0)
 			(hide yes)
@@
 			)
 		)
-		(property "Footprint" "willkeebs_keyboard:NF_LED_1206_SW_KS33_3_0_HS_1U"
+		(property "Footprint" "willkeebs_keyboard:KS-33B Hotswap 1u"
 			(at 217.17 86.36 0)
 			(hide yes)
@@
 			)
 		)
-		(property "Footprint" "willkeebs_keyboard:NF_LED_1206_SW_KS33_3_0_HS_1U"
+		(property "Footprint" "willkeebs_keyboard:KS-33B Hotswap 1u"
 			(at 273.05 71.12 0)
 			(hide yes)
@@
 			)
 		)
-		(property "Footprint" "willkeebs_keyboard:NF_LED_1206_SW_KS33_3_0_HS_1U"
+		(property "Footprint" "willkeebs_keyboard:KS-33B Hotswap 1u"
 			(at 259.08 71.12 0)
 			(hide yes)
@@
 			)
 		)
-		(property "Footprint" "willkeebs_keyboard:NF_LED_1206_SW_KS33_3_0_HS_1U"
+		(property "Footprint" "willkeebs_keyboard:KS-33B Hotswap 1u"
 			(at 245.11 57.15 0)
 			(hide yes)
@@
 			)
 		)
-		(property "Footprint" "willkeebs_keyboard:NF_LED_1206_SW_KS33_3_0_HS_1U"
+		(property "Footprint" "willkeebs_keyboard:KS-33B Hotswap 1u"
 			(at 245.11 41.91 0)
 			(hide yes)
@@
 			)
 		)
-		(property "Footprint" "willkeebs_keyboard:NF_LED_1206_SW_KS33_3_0_HS_1U"
+		(property "Footprint" "willkeebs_keyboard:KS-33B Hotswap 1u"
 			(at 273.05 57.15 0)
 			(hide yes)
@@
 			)
 		)
-		(property "Footprint" "willkeebs_keyboard:NF_LED_1206_SW_KS33_3_0_HS_1U"
+		(property "Footprint" "willkeebs_keyboard:KS-33B Hotswap 1u"
 			(at 245.11 71.12 0)
 			(hide yes)
@@
 			)
 		)
-		(property "Footprint" "willkeebs_keyboard:NF_LED_1206_SW_KS33_3_0_HS_1U"
+		(property "Footprint" "willkeebs_keyboard:KS-33B Hotswap 1u"
 			(at 287.02 71.12 0)
 			(hide yes)
@@
 			)
 		)
-		(property "Footprint" "willkeebs_keyboard:NF_LED_1206_SW_KS33_3_0_HS_1U"
+		(property "Footprint" "willkeebs_keyboard:KS-33B Hotswap 1u"
 			(at 217.17 41.91 0)
 			(hide yes)
@@
 			)
 		)
-		(property "Footprint" "willkeebs_keyboard:NF_LED_1206_SW_KS33_3_0_HS_1U"
+		(property "Footprint" "willkeebs_keyboard:KS-33B Hotswap 1u"
 			(at 217.17 71.12 0)
 			(hide yes)
@@
 			)
 		)
-		(property "Footprint" "willkeebs_keyboard:NF_LED_1206_SW_KS33_3_0_HS_1U"
+		(property "Footprint" "willkeebs_keyboard:KS-33B Hotswap 1u"
 			(at 245.11 86.36 0)
 			(hide yes)
@@
 			)
 		)
-		(property "Footprint" "willkeebs_keyboard:NF_LED_1206_SW_KS33_3_0_HS_1U"
+		(property "Footprint" "willkeebs_keyboard:KS-33B Hotswap 1u"
 			(at 273.05 41.91 0)
 			(hide yes)
@@
 			)
 		)
-		(property "Footprint" "willkeebs_keyboard:NF_LED_1206_SW_KS33_3_0_HS_1U"
+		(property "Footprint" "willkeebs_keyboard:KS-33B Hotswap 1u"
 			(at 231.14 71.12 0)
 			(hide yes)
@@
 			)
 		)
-		(property "Footprint" "willkeebs_keyboard:NF_LED_1206_SW_KS33_3_0_HS_1U"
+		(property "Footprint" "willkeebs_keyboard:KS-33B Hotswap 1u"
 			(at 287.02 57.15 0)
 			(hide yes)
@@
 			)
 		)
-		(property "Footprint" "willkeebs_keyboard:NF_LED_1206_SW_KS33_3_0_HS_1U"
+		(property "Footprint" "willkeebs_keyboard:KS-33B Hotswap 1u"
 			(at 231.14 86.36 0)
 			(hide yes)
@@
 			)
 		)
-		(property "Footprint" "willkeebs_keyboard:NF_LED_1206_SW_KS33_3_0_HS_1U"
+		(property "Footprint" "willkeebs_keyboard:KS-33B Hotswap 1u"
 			(at 217.17 57.15 0)
 			(hide yes)
@@
 			)
 		)
-		(property "Footprint" "willkeebs_keyboard:NF_LED_1206_SW_KS33_3_0_HS_1U"
+		(property "Footprint" "willkeebs_keyboard:KS-33B Hotswap 1u"
 			(at 259.08 41.91 0)
 			(hide yes)
@@
 			)
 		)
-		(property "Footprint" "willkeebs_keyboard:NF_LED_1206_SW_KS33_3_0_HS_1U"
+		(property "Footprint" "willkeebs_keyboard:KS-33B Hotswap 1u"
 			(at 231.14 57.15 0)
 			(hide yes)

Commit message: feat: remove unused components from BOM and POS
Parts:
- BT2_R1, TP4, TP4_R1, TP5, TP6_R1: now left out of the parts list
Changed lines of the file:
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@@
 		(body_style 1)
 		(exclude_from_sim no)
-		(in_bom yes)
+		(in_bom no)
 		(on_board yes)
-		(in_pos_files yes)
+		(in_pos_files no)
 		(dnp no)
 		(property "Reference" "BT2_R1"
@@
 		(body_style 1)
 		(exclude_from_sim no)
-		(in_bom yes)
+		(in_bom no)
 		(on_board yes)
-		(in_pos_files yes)
+		(in_pos_files no)
 		(dnp no)
 		(property "Reference" "TP4"
@@
 		(body_style 1)
 		(exclude_from_sim no)
-		(in_bom yes)
+		(in_bom no)
 		(on_board yes)
-		(in_pos_files yes)
+		(in_pos_files no)
 		(dnp no)
 		(fields_autoplaced yes)
@@
 		(body_style 1)
 		(exclude_from_sim no)
-		(in_bom yes)
+		(in_bom no)
 		(on_board yes)
-		(in_pos_files yes)
+		(in_pos_files no)
 		(dnp no)
 		(property "Reference" "TP6_R1"
@@
 		(body_style 1)
 		(exclude_from_sim no)
-		(in_bom yes)
+		(in_bom no)
 		(on_board yes)
-		(in_pos_files yes)
+		(in_pos_files no)
 		(dnp no)
 		(property "Reference" "TP4_R1"

Commit message: feat: remove unused components from BOM and POS
Parts:
- LOGO_R1: now left out of the parts list
Changed lines of the file:
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@@
 		(body_style 1)
 		(exclude_from_sim no)
-		(in_bom yes)
+		(in_bom no)
 		(on_board yes)
-		(in_pos_files yes)
+		(in_pos_files no)
 		(dnp no)
 		(fields_autoplaced yes)
